File: A7105 reference design.brd (EAGLE design)
At the start: 13.5 x 11.5 mm, 39 parts, among them U1 A7105, U2 STM32F031G4U6, X1 ECX-2236

Commit message: STM work
Parts:
- removed C19: 1uF, Perfect_0402:0402
- removed R5: 200, Perfect_0402:0402
- removed U$5: SMD-CHIP-LED-0402, alienflight:0402LED
- added C21: 4.7uF, Perfect_0402:0402
- added C22: 10000pF, Perfect_0402:0402
- added C23: 1uF, Perfect_0402:0402
- added LED1: RGBLED_CANODE, nikdavis:SML-LX0404SIUPGUSB
- added R3, R4, R7: 200, Perfect_0402:0402
- moved C20 6.42 mm to (13.8, 12.8), flipped to the top
- moved TP1 1.82 mm to (11.0, 9.73)
- moved TP2 1.37 mm to (12.6, 9.73)
- moved TP3 0.81 mm to (9.47, 9.73)
- moved R6 0.23 mm to (11.1, 4.12), flipped to the top
- moved R2 0.23 mm to (12.2, 7.13), flipped to the top
- flipped C18 to the top
Connections:
- net N$11 renamed NRST
- net N$5 renamed BOOT0
- removed net N$9: R5.2, U$5.2
- removed net STATUS: R5.1
- new net LED_B: R7.1, U2.15
- new net LED_G: R4.1, U2.14
- new net LED_R: R3.1, U2.13
- new net N$15: LED1.P$2, R3.2
- new net N$16: LED1.P$4, R4.2
- new net N$17: LED1.P$3, R7.2
- net GND: now also C21.2, C22.2, C23.2; no longer C19.2, U$5.1
- net MCUCLK: now also U2.2
- net VCC: now also C21.1, C22.1, C23.1, LED1.P$1; no longer C19.1
Routing:
- net MCUCLK: track 0.00 -> 7.06 mm, vias 0 -> 1
- net SBUS: track 0.00 -> 4.24 mm, vias 0 -> 1
- net SCK: track 8.43 -> 4.94 mm
- net SCS: track 10.0 -> 6.63 mm
- net SWD: track 2.62 -> 0.00 mm, vias 1 -> 0
- net SWCLK: track 1.86 -> 0.00 mm, vias 1 -> 0
- net NRST: track 0.00 -> 1.31 mm, vias 0 -> 1
- net BOOT0: track 0.00 -> 1.20 mm, vias 0 -> 1
- net MOSI: track 1.25 -> 1.51 mm, vias 0 -> 1
Other:
- board text removed: "MI"
- board text removed: "MO"
- board text removed: "RST"
- board text removed: "SCK"

Commit message: STM "ready"
Parts:
- moved C22 7.91 mm to (10.4, 2.97), flipped to the bottom, turned to 180 degrees
- moved C23 7.02 mm to (10.4, 3.84), flipped to the bottom, turned to 180 degrees
- moved C20 5.15 mm to (9.47, 10.1), flipped to the bottom, turned to 180 degrees
- moved R7 4.98 mm to (5.74, 8.86), turned to 0 degrees
- moved R4 4.59 mm to (5.89, 8.00)
- moved C21 4.35 mm to (11.3, 10.2), flipped to the bottom, turned to 180 degrees
- moved R3 0.65 mm to (8.43, 8.31), turned to 137.7 degrees
- moved R6 0.36 mm to (10.8, 4.12)
- moved U$6 0.23 mm to (12.1, 2.83)
- moved U$9 0.18 mm to (10.5, 1.18)
- moved U$8 0.16 mm to (12.1, 1.18)
- moved R2 0.14 mm to (12.1, 7.02)
Connections:
- net GPIO1: now also U2.11; no longer U2.20
Routing:
- net VCC: track 1.61 -> 34.4 mm, vias 0 -> 4
- net N$16: track 0.00 -> 4.69 mm, vias 0 -> 1
- net GND: track 3.82 -> 8.34 mm, vias 17 -> 23
- net N$17: track 0.00 -> 3.83 mm, vias 0 -> 1
- net SWCLK: track 0.00 -> 2.16 mm, vias 0 -> 1
- net LED_R: track 0.00 -> 2.09 mm, vias 0 -> 1
- net LED_B: track 0.00 -> 1.82 mm
- net GPIO1: track 0.00 -> 1.67 mm, vias 0 -> 1
- net LED_G: track 0.00 -> 1.35 mm
- net SWD: track 0.00 -> 1.19 mm, vias 0 -> 1
- net N$15: track 0.00 -> 1.00 mm
- net MCUCLK: track 7.06 -> 7.89 mm, vias 1 -> 2
- net SDIO: track 6.37 -> 5.76 mm
- net MOSI: track 1.51 -> 0.95 mm
Other:
- board size 13.5 x 11.5 mm -> 13.4 x 11.1 mm
