File: A7105 reference design.sch (EAGLE design)
At the start: 42 parts, among them U1 A7105, U2 STM32F031G4U6, U3 NMOSSOT833B/1006, X1 ECX-2236

Commit message: First steps
Remove inverter
Make todo list
Parts:
- removed R3, R4: 10k, Perfect_0402:RES_0402
- removed U3: NMOSSOT833B/1006, nikdavis:NMOSSOT833B/1006
Connections:
- removed net G: R4.2, U3.G
- removed net NSBUS: R4.1, U2.PB6
- net GND: no longer U3.S
- net SBUS: now also U2.PB6; no longer R3.1, U3.D
- net VCC: no longer R3.2
Other:
- note added: "NEED: - led pin - gpio pin (pick one with edge interrupts close to a7105) - uart tx for sbus - CHECK all pins -- i'm pretty sure they're wrong - extra LED? - analog pin for battery (requires step down resistors ugh) - GPIO exposed (can be anywhere) - spi test pads (even if tiny) - clock input (maybe not necessary but I can route still)"
- note removed: "NEED: - led pin - gpio pin (pick one with edge interrupts close to a7105) - uart tx for sbus"
Changed lines of the file:
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@@
 <part name="GND7" library="SparkFun-PowerSymbols" deviceset="GND" device=""/>
 <part name="R2" library="Perfect_0402" deviceset="RES_0402" device="" value="10k"/>
-<part name="R3" library="Perfect_0402" deviceset="RES_0402" device="" value="10k"/>
 <part name="SUPPLY2" library="SparkFun-PowerSymbols" deviceset="VCC" device=""/>
-<part name="GND5" library="SparkFun-PowerSymbols" deviceset="GND" device=""/>
-<part name="R4" library="Perfect_0402" deviceset="RES_0402" device="" value="10k"/>
 <part name="R5" library="Perfect_0402" deviceset="RES_0402" device="" value="200"/>
 <part name="U$5" library="alienflight" deviceset="SMD-CHIP-LED-0402" device=""/>
@@
 <part name="U$8" library="AlienWhoop" deviceset="TESTPAD" device=""/>
 <part name="U$9" library="AlienWhoop" deviceset="TESTPAD" device=""/>
-<part name="U3" library="nikdavis" deviceset="NMOS" device="SOT833B/1006"/>
 <part name="GND11" library="SparkFun-PowerSymbols" deviceset="GND" device=""/>
 <part name="C19" library="Perfect_0402" deviceset="CAP_0402" device="" value="1uF"/>
@@
 <text x="101.6" y="-40.64" size="3.048" layer="94">Nikolas Davis</text>
 <text x="180.34" y="-40.64" size="3.048" layer="94">0.1</text>
-<text x="88.9" y="5.08" size="1.778" layer="91">NEED:
+<text x="86.36" y="-7.62" size="1.778" layer="91">NEED:
 - led pin
 - gpio pin (pick one with edge interrupts close to a7105)
-- uart tx for sbus</text>
+- uart tx for sbus
+- CHECK all pins -- i'm pretty sure they're wrong
+- extra LED?
+- analog pin for battery (requires step down resistors ugh)
+- GPIO exposed (can be anywhere)
+- spi test pads (even if tiny)
+- clock input (maybe not necessary but I can route still)
+</text>
 </plain>
 <instances>
@@
 <attribute name="VALUE" x="133.35" y="47.498" size="1.778" layer="96"/>
 </instance>
-<instance part="R3" gate="G$1" x="132.08" y="119.38" smashed="yes" rot="R90">
-<attribute name="NAME" x="130.5814" y="120.65" size="1.778" layer="95" rot="R90"/>
-<attribute name="VALUE" x="135.382" y="120.65" size="1.778" layer="96" rot="R90"/>
-</instance>
-<instance part="SUPPLY2" gate="G$1" x="132.08" y="132.08" smashed="yes">
-<attribute name="VALUE" x="132.08" y="134.874" size="1.778" layer="96" align="bottom-center"/>
-</instance>
-<instance part="GND5" gate="1" x="132.08" y="101.6" smashed="yes">
-<attribute name="VALUE" x="132.08" y="101.346" size="1.778" layer="96" align="top-center"/>
-</instance>
-<instance part="R4" gate="G$1" x="111.76" y="109.22" smashed="yes">
-<attribute name="NAME" x="113.03" y="110.7186" size="1.778" layer="95"/>
-<attribute name="VALUE" x="113.03" y="105.918" size="1.778" layer="96"/>
+<instance part="SUPPLY2" gate="G$1" x="142.24" y="127" smashed="yes">
+<attribute name="VALUE" x="142.24" y="129.794" size="1.778" layer="96" align="bottom-center"/>
 </instance>
 <instance part="R5" gate="G$1" x="185.42" y="30.48" smashed="yes" rot="R270">
@@
 <instance part="U$8" gate="G$1" x="167.64" y="119.38" smashed="yes"/>
 <instance part="U$9" gate="G$1" x="167.64" y="116.84" smashed="yes"/>
-<instance part="U3" gate="G$1" x="129.54" y="111.76" smashed="yes">
-<attribute name="NAME" x="134.62" y="111.76" size="1.778" layer="95" font="vector"/>
-</instance>
 <instance part="GND11" gate="1" x="160.02" y="104.14" smashed="yes">
 <attribute name="VALUE" x="160.02" y="103.886" size="1.778" layer="96" align="top-center"/>
@@
 </segment>
 <segment>
-<pinref part="GND5" gate="1" pin="GND"/>
-<wire x1="132.08" y1="104.14" x2="132.08" y2="106.68" width="0.1524" layer="91"/>
-<pinref part="U3" gate="G$1" pin="S"/>
-</segment>
-<segment>
 <pinref part="U$5" gate="G$1" pin="C"/>
 <pinref part="GND10" gate="1" pin="GND"/>
@@
 <wire x1="43.18" y1="0" x2="43.18" y2="-5.08" width="0.1524" layer="91"/>
 <pinref part="C9" gate="G$1" pin="1"/>
-</segment>
-<segment>
-<pinref part="R3" gate="G$1" pin="2"/>
-<pinref part="SUPPLY2" gate="G$1" pin="VCC"/>
-<wire x1="132.08" y1="129.54" x2="132.08" y2="132.08" width="0.1524" layer="91"/>
-<wire x1="132.08" y1="129.54" x2="139.7" y2="129.54" width="0.1524" layer="91"/>
-<junction x="132.08" y="129.54"/>
-<wire x1="139.7" y1="129.54" x2="139.7" y2="119.38" width="0.1524" layer="91"/>
-<wire x1="139.7" y1="119.38" x2="154.94" y2="119.38" width="0.1524" layer="91"/>
-<label x="149.86" y="119.38" size="1.778" layer="95"/>
-<pinref part="U$8" gate="G$1" pin="1"/>
-<pinref part="C19" gate="G$1" pin="1"/>
-<wire x1="154.94" y1="119.38" x2="162.56" y2="119.38" width="0.1524" layer="91"/>
-<wire x1="154.94" y1="119.38" x2="154.94" y2="116.84" width="0.1524" layer="91"/>
-<junction x="154.94" y="119.38"/>
 </segment>
 <segment>
@@
 <wire x1="121.92" y1="68.58" x2="121.92" y2="71.12" width="0.1524" layer="91"/>
 <junction x="121.92" y="71.12"/>
+</segment>
+<segment>
+<label x="149.86" y="119.38" size="1.778" layer="95"/>
+<pinref part="U$8" gate="G$1" pin="1"/>
+<pinref part="C19" gate="G$1" pin="1"/>
+<wire x1="142.24" y1="119.38" x2="154.94" y2="119.38" width="0.1524" layer="91"/>
+<wire x1="154.94" y1="119.38" x2="162.56" y2="119.38" width="0.1524" layer="91"/>
+<wire x1="154.94" y1="119.38" x2="154.94" y2="116.84" width="0.1524" layer="91"/>
+<junction x="154.94" y="119.38"/>
+<pinref part="SUPPLY2" gate="G$1" pin="VCC"/>
+<wire x1="142.24" y1="127" x2="142.24" y2="119.38" width="0.1524" layer="91"/>
+<junction x="142.24" y="119.38"/>
 </segment>
 </net>
@@
 </segment>
 </net>
-<net name="NSBUS" class="0">
-<segment>
-<pinref part="R4" gate="G$1" pin="1"/>
-<wire x1="96.52" y1="109.22" x2="111.76" y2="109.22" width="0.1524" layer="91"/>
-<label x="96.52" y="109.22" size="1.778" layer="95"/>
+<net name="SBUS" class="0">
+<segment>
+<wire x1="144.78" y1="121.92" x2="162.56" y2="121.92" width="0.1524" layer="91"/>
+<label x="149.86" y="121.92" size="1.778" layer="95"/>
+<pinref part="U$6" gate="G$1" pin="1"/>
 </segment>
 <segment>
@@
 <wire x1="119.38" y1="48.26" x2="129.54" y2="48.26" width="0.1524" layer="91"/>
 <label x="124.46" y="48.26" size="1.778" layer="95"/>
-</segment>
-</net>
-<net name="SBUS" class="0">
-<segment>
-<pinref part="R3" gate="G$1" pin="1"/>
-<wire x1="132.08" y1="116.84" x2="132.08" y2="119.38" width="0.1524" layer="91"/>
-<wire x1="132.08" y1="119.38" x2="137.16" y2="119.38" width="0.1524" layer="91"/>
-<junction x="132.08" y="119.38"/>
-<wire x1="137.16" y1="119.38" x2="137.16" y2="121.92" width="0.1524" layer="91"/>
-<wire x1="137.16" y1="121.92" x2="162.56" y2="121.92" width="0.1524" layer="91"/>
-<label x="149.86" y="121.92" size="1.778" layer="95"/>
-<pinref part="U$6" gate="G$1" pin="1"/>
-<pinref part="U3" gate="G$1" pin="D"/>
-</segment>
-</net>
-<net name="G" class="0">
-<segment>
-<pinref part="R4" gate="G$1" pin="2"/>
-<wire x1="121.92" y1="109.22" x2="124.46" y2="109.22" width="0.1524" layer="91"/>
-<pinref part="U3" gate="G$1" pin="G"/>
 </segment>
 </net>
@@
 which will not be processed correctly with this version.
 </note>
-<note version="8.3" severity="warning">
-Since Version 8.3, EAGLE supports URNs for individual library
-assets (packages, symbols, and devices). The URNs of those assets
-will not be understood (or retained) with this version.
-</note>
 </compatibility>

Commit message: STM work
Parts:
- removed C19: 1uF, Perfect_0402:CAP_0402
- removed R5: 200, Perfect_0402:RES_0402
- removed U$5: SMD-CHIP-LED-0402, alienflight:SMD-CHIP-LED-0402
- added C21: 4.7uF, Perfect_0402:CAP_0402
- added C22: 10000pF, Perfect_0402:CAP_0402
- added C23: 1uF, Perfect_0402:CAP_0402
- added LED1: RGBLED_CANODE, nikdavis:RGBLED_CANODE
- added R3, R4, R7: 200, Perfect_0402:RES_0402
Connections:
- net N$11 renamed NRST
- net N$5 renamed BOOT0
- removed net N$9: R5.2, U$5.A
- removed net STATUS: R5.1
- new net LED_B: R7.1, U2.PB1
- new net LED_G: R4.1, U2.PB0
- new net LED_R: R3.1, U2.PA7
- new net N$15: LED1.R_P2, R3.2
- new net N$16: LED1.G_P4, R4.2
- new net N$17: LED1.B_P3, R7.2
- net GND: now also C21.2, C22.2, C23.2; no longer C19.2, U$5.C
- net MCUCLK: now also U2.PF0
- net VCC: now also C21.1, C22.1, C23.1, LED1.AN_P1; no longer C19.1
Other:
- note added: "NEED: - led pin - gpio pin (pick one with edge interrupts close to a7105) - uart tx for sbus - CHECK all pins -- i'm pretty sure they're wrong - extra LED? - analog pin for battery (requires step down resistors ugh) & VDDA cap - GPIO exposed (can be anywhere) - spi test pads (even if tiny) - clock input (maybe not necessary but I can route still)"
- note added: "VDD"
- note added: "VDDA"
- note added: "verified sbus spi clk boot decoup led current"
- note removed: "NEED: - led pin - gpio pin (pick one with edge interrupts close to a7105) - uart tx for sbus - CHECK all pins -- i'm pretty sure they're wrong - extra LED? - analog pin for battery (requires step down resistors ugh) - GPIO exposed (can be anywhere) - spi test pads (even if tiny) - clock input (maybe not necessary but I can route still)"

Commit message: STM "ready"
Connections:
- net GPIO1: now also U2.PA5; no longer U2.PA10
Changed lines of the file:
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@@
 </segment>
 <segment>
-<pinref part="U2" gate="G$1" pin="PA10"/>
-<wire x1="88.9" y1="35.56" x2="78.74" y2="35.56" width="0.1524" layer="91"/>
-<label x="78.74" y="35.56" size="1.778" layer="95"/>
+<pinref part="U2" gate="G$1" pin="PA5"/>
+<wire x1="88.9" y1="48.26" x2="78.74" y2="48.26" width="0.1524" layer="91"/>
+<label x="78.74" y="48.26" size="1.778" layer="95"/>
 </segment>
 </net>
